File: EEE3099S_CircuitDesign_Group1.kicad_sch (KiCad schematic)
At the start: 21 parts, among them IC1 L298N, M1 Motor_DC, M2 Motor_DC, SW1 SW_Push, U1 ABX00027, U3 HC-SR04, U9 ONBOARD_HBridge_ 5V_REGULATOR

Commit message: Repo Update
Connections:
- net NANO_D10: now also U8. (LV4); no longer U4. (LV4)
- net NANO_D10_5V: now also U8. (LV4); no longer U4. (LV4)
- net NANO_D11: now also U8. (LV4); no longer U4. (LV4)
- net NANO_D11_5V: now also U8. (LV4); no longer U4. (LV4)
- net NANO_D6: now also U4. (LV4); no longer U8. (LV4)
- net NANO_D6_HV: now also U4. (LV4); no longer U8. (LV4)
- net NANO_20: now reaches U1.10 (A6)
- net NANO_20: now also U6. (Vcc)
- net NANO_D21: now reaches U1.11 (A7)
- net NANO_D21: now also U7. (Vcc)
- net NANO_D15: now reaches U1.5 (A1)
- net NANO_D15: now also U2. (Vcc)
- net NANO_D18: now reaches U1.7 (A3)
- net NANO_D18: now also U5. (Vcc)
- net NANO_D2: no longer names the net of U1.20 (D2)
- net NANO_D2: no longer U2. (Vcc)
- net NANO_D3: no longer names the net of U1.21 (D3/PWM)
- net NANO_D3: no longer U5. (Vcc)
- net NANO_D4: no longer names the net of U1.22 (D4)
- net NANO_D4: no longer U6. (Vcc)
- net NANO_D5: no longer names the net of U1.23 (D5/PWM)
- net NANO_D5: no longer U7. (Vcc)
Changed lines of the file:
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@@
   (junction (at 77.47 152.4) (diameter 0) (color 0 0 0 0)
   )
-  (no_connect (at 114.3 125.73))
   (no_connect (at 71.12 39.37))
-  (no_connect (at 187.96 119.38))
   (no_connect (at 71.12 54.61))
-  (no_connect (at 114.3 135.89))
+  (no_connect (at 149.86 113.03))
   (no_connect (at 114.3 113.03))
+  (no_connect (at 179.07 138.43))
+  (no_connect (at 212.09 138.43))
   (no_connect (at 114.3 130.81))
-  (no_connect (at 114.3 128.27))
   (no_connect (at 114.3 123.19))
-  (no_connect (at 203.2 119.38))
-  (no_connect (at 114.3 120.65))
   (no_connect (at 114.3 140.97))
+  (no_connect (at 149.86 115.57))
   (no_connect (at 114.3 143.51))
   (no_connect (at 149.86 102.87))
-  (no_connect (at 114.3 133.35))
   (no_connect (at 142.24 54.61))
+  (no_connect (at 114.3 128.27))
+  (no_connect (at 149.86 118.11))
+  (no_connect (at 149.86 110.49))
   (wire (pts (xy 149.86 105.41) (xy 154.94 105.41))
     (stroke (width 0) (type default))
@@
     (effects (font (size 1.27 1.27)) (justify right bottom))
   )
+  (label "NANO_D18" (at 114.3 125.73 180) (fields_autoplaced)
+    (effects (font (size 1.27 1.27)) (justify right bottom))
+  )
   (label "NANO_D13_5V" (at 203.2 109.22 0) (fields_autoplaced)
     (effects (font (size 1.27 1.27)) (justify left bottom))
@@
     (effects (font (size 1.27 1.27)) (justify left bottom))
   )
-  (label "NANO_D3" (at 149.86 113.03 0) (fields_autoplaced)
-    (effects (font (size 1.27 1.27)) (justify left bottom))
-  )
-  (label "NANO_D11_5V" (at 212.09 138.43 0) (fields_autoplaced)
+  (label "NANO_D6_HV" (at 212.09 135.89 0) (fields_autoplaced)
     (effects (font (size 1.27 1.27)) (justify left bottom))
   )
@@
     (effects (font (size 1.27 1.27)) (justify left bottom))
   )
-  (label "NANO_D2" (at 193.04 29.21 180) (fields_autoplaced)
-    (effects (font (size 1.27 1.27)) (justify right bottom))
-  )
-  (label "NANO_D4" (at 193.04 48.26 180) (fields_autoplaced)
-    (effects (font (size 1.27 1.27)) (justify right bottom))
-  )
-  (label "NANO_D4" (at 149.86 115.57 0) (fields_autoplaced)
-    (effects (font (size 1.27 1.27)) (justify left bottom))
+  (label "NANO_20" (at 193.04 48.26 180) (fields_autoplaced)
+    (effects (font (size 1.27 1.27)) (justify right bottom))
+  )
+  (label "NANO_D11" (at 179.07 116.84 180) (fields_autoplaced)
+    (effects (font (size 1.27 1.27)) (justify right bottom))
+  )
+  (label "NANO_D10" (at 187.96 119.38 180) (fields_autoplaced)
+    (effects (font (size 1.27 1.27)) (justify right bottom))
   )
   (label "M1_GND" (at 118.11 73.66 270) (fields_autoplaced)
     (effects (font (size 1.27 1.27)) (justify right bottom))
   )
+  (label "NANO_D8_5V" (at 203.2 128.27 0) (fields_autoplaced)
+    (effects (font (size 1.27 1.27)) (justify left bottom))
+  )
   (label "NANO_D8" (at 149.86 125.73 0) (fields_autoplaced)
     (effects (font (size 1.27 1.27)) (justify left bottom))
   )
-  (label "NANO_D5" (at 149.86 118.11 0) (fields_autoplaced)
-    (effects (font (size 1.27 1.27)) (justify left bottom))
-  )
-  (label "NANO_D5" (at 209.55 48.26 180) (fields_autoplaced)
+  (label "NANO_D15" (at 193.04 29.21 180) (fields_autoplaced)
+    (effects (font (size 1.27 1.27)) (justify right bottom))
+  )
+  (label "NANO_D21" (at 209.55 48.26 180) (fields_autoplaced)
     (effects (font (size 1.27 1.27)) (justify right bottom))
   )
@@
     (effects (font (size 1.27 1.27)) (justify right bottom))
   )
-  (label "NANO_D8" (at 179.07 135.89 180) (fields_autoplaced)
+  (label "NANO_D21" (at 114.3 135.89 180) (fields_autoplaced)
     (effects (font (size 1.27 1.27)) (justify right bottom))
   )
@@
     (effects (font (size 1.27 1.27)) (justify left bottom))
   )
-  (label "NANO_D11" (at 179.07 138.43 180) (fields_autoplaced)
-    (effects (font (size 1.27 1.27)) (justify right bottom))
-  )
-  (label "NANO_D6" (at 179.07 116.84 180) (fields_autoplaced)
-    (effects (font (size 1.27 1.27)) (justify right bottom))
-  )
   (label "NANO_D6_HV" (at 201.93 69.85 180) (fields_autoplaced)
     (effects (font (size 1.27 1.27)) (justify right bottom))
@@
     (effects (font (size 1.27 1.27)) (justify left bottom))
   )
-  (label "NANO_D6_HV" (at 212.09 116.84 0) (fields_autoplaced)
-    (effects (font (size 1.27 1.27)) (justify left bottom))
-  )
-  (label "NANO_D2" (at 149.86 110.49 0) (fields_autoplaced)
+  (label "NANO_D8" (at 187.96 128.27 180) (fields_autoplaced)
+    (effects (font (size 1.27 1.27)) (justify right bottom))
+  )
+  (label "NANO_D10_5V" (at 203.2 119.38 0) (fields_autoplaced)
     (effects (font (size 1.27 1.27)) (justify left bottom))
   )
@@
     (effects (font (size 1.27 1.27)) (justify right bottom))
   )
+  (label "NANO_D11_5V" (at 212.09 116.84 0) (fields_autoplaced)
+    (effects (font (size 1.27 1.27)) (justify left bottom))
+  )
   (label "NANO_D9" (at 187.96 125.73 180) (fields_autoplaced)
     (effects (font (size 1.27 1.27)) (justify right bottom))
@@
     (effects (font (size 1.27 1.27)) (justify left bottom))
   )
-  (label "NANO_D10" (at 187.96 128.27 180) (fields_autoplaced)
-    (effects (font (size 1.27 1.27)) (justify right bottom))
-  )
-  (label "NANO_D3" (at 209.55 29.21 180) (fields_autoplaced)
+  (label "NANO_D6" (at 179.07 135.89 180) (fields_autoplaced)
+    (effects (font (size 1.27 1.27)) (justify right bottom))
+  )
+  (label "NANO_D18" (at 209.55 29.21 180) (fields_autoplaced)
     (effects (font (size 1.27 1.27)) (justify right bottom))
   )
@@
     (effects (font (size 1.27 1.27)) (justify left bottom))
   )
-  (label "NANO_D8_5V" (at 212.09 135.89 0) (fields_autoplaced)
-    (effects (font (size 1.27 1.27)) (justify left bottom))
-  )
   (label "NANO_D9_5V" (at 71.12 49.53 180) (fields_autoplaced)
     (effects (font (size 1.27 1.27)) (justify right bottom))
@@
     (effects (font (size 1.27 1.27)) (justify left bottom))
   )
-  (label "NANO_D10_5V" (at 203.2 128.27 0) (fields_autoplaced)
-    (effects (font (size 1.27 1.27)) (justify left bottom))
-  )
   (label "NANO_D9" (at 149.86 128.27 0) (fields_autoplaced)
     (effects (font (size 1.27 1.27)) (justify left bottom))
   )
+  (label "NANO_20" (at 114.3 133.35 180) (fields_autoplaced)
+    (effects (font (size 1.27 1.27)) (justify right bottom))
+  )
+  (label "NANO_D15" (at 114.3 120.65 180) (fields_autoplaced)
+    (effects (font (size 1.27 1.27)) (justify right bottom))
+  )
   (label "NANO_D10_5V" (at 142.24 41.91 0) (fields_autoplaced)
